Commit message: GZ SIM, 3D Lidar 추가

File: linorobot2_description/urdf/4wd_properties.urdf.xacro (robot description, xacro)
@@ -24,3 +24,6 @@
     <origin xyz="-0.065 0 0.255" rpy="0 0 0"/>
   </xacro:property>
+  <xacro:property name="mid360_pose">
+    <origin xyz="0 0 0.300" rpy="0 0 0"/>
+  </xacro:property>
 </robot>

File: linorobot2_description/urdf/robots/4wd.urdf.xacro (robot description, xacro)
@@ -9,4 +9,5 @@
   <xacro:include filename="$(find linorobot2_description)/urdf/sensors/depth_sensor.urdf.xacro" />
   <xacro:include filename="$(find linorobot2_description)/urdf/controllers/skid_steer.urdf.xacro" />
+  <xacro:include filename="$(find linorobot2_description)/urdf/sensors/lidar_mid360_sensor.urdf.xacro" />
   <xacro:base
     length="${base_length}"
@@ -65,4 +66,7 @@
     <xacro:insert_block name="depth_sensor_pose" />
   </xacro:depth_sensor>
+  <xacro:lidar3d_sensor>
+    <xacro:insert_block name="mid360_pose" />
+  </xacro:lidar3d_sensor>
   <xacro:diff_drive_controller
     wheel_separation="${wheel_pos_y * 2}"

Commit message: Added,ros2 livox simulation for gazebo classic

File: linorobot2_description/urdf/4wd_properties.urdf.xacro (robot description, xacro)
@@ -21,3 +21,6 @@
     <origin xyz="-0.2375 0.0 0.255" rpy="0 0 3.14159"/>
   </xacro:property>
+  <xacro:property name="mid360_pose">
+    <origin xyz="0 0 0.300" rpy="0 0 0"/>
+  </xacro:property>
 </robot>

File: linorobot2_description/urdf/robots/4wd.urdf.xacro (robot description, xacro)
@@ -9,4 +9,5 @@
   <xacro:include filename="$(find linorobot2_description)/urdf/sensors/camera.urdf.xacro" />
   <xacro:include filename="$(find linorobot2_description)/urdf/controllers/skid_steer.urdf.xacro" />
+  <xacro:include filename="$(find ros2_livox_simulation)/urdf/mid360.xacro" />
   <xacro:base
     length="${base_length}"
@@ -66,4 +67,7 @@
     <xacro:insert_block name="rear_camera_sensor_pose" />
   </xacro:rgb_camera>
+  <xacro:mid360 name="livox" parent="base_link" topic="mid360">
+    <xacro:insert_block name="mid360_pose"/>
+  </xacro:mid360>
   <xacro:diff_drive_controller
     wheel_separation="${wheel_pos_y * 2}"
