Commit message: mapless slam + gps하고있는데 잘 안됨 ㅠㅠ

File: linorobot2_description/urdf/controllers/skid_steer.urdf.xacro (robot description, xacro)
@@ -3,7 +3,7 @@
     <gazebo>
       <plugin name="differential_drive_controller" filename="libgazebo_ros_diff_drive.so">
-        <ros>
+        <!-- <ros>
           <remapping>odom:=odom/unfiltered</remapping>
-        </ros>
+        </ros> -->
         <num_wheel_pairs>2</num_wheel_pairs>
         <left_joint>front_left_wheel_joint</left_joint>
@@ -17,9 +17,9 @@
         <updateRate>100</updateRate>
         <max_wheel_acceleration>1.0</max_wheel_acceleration>
-        <robot_base_frame>base_footprint</robot_base_frame>
-        <publish_odom>true</publish_odom>
+        <robot_base_frame>base_link</robot_base_frame>
+        <publish_odom>false</publish_odom>
         <publish_odom_tf>false</publish_odom_tf>
-        <publish_wheel_tf>true</publish_wheel_tf>
-        <odometry_frame>odom</odometry_frame>
+        <publish_wheel_tf>false</publish_wheel_tf>
+        <odometry_frame>odom_gazebo</odometry_frame>
       </plugin>
     </gazebo>

File: linorobot2_description/urdf/robots/4wd.urdf.xacro (robot description, xacro)
@@ -9,4 +9,5 @@
   <xacro:include filename="$(find linorobot2_description)/urdf/sensors/camera.urdf.xacro" />
   <xacro:include filename="$(find linorobot2_description)/urdf/sensors/lidar.xacro" />
+  <xacro:include filename="$(find linorobot2_description)/urdf/sensors/gps.urdf.xacro" />
   <!-- vlp-16 -->
   <xacro:include filename="$(find linorobot2_description)/urdf/controllers/skid_steer.urdf.xacro" />
@@ -77,3 +78,15 @@
     wheel_torque="${wheel_torque}"
   />
+  <link name="camera_init"/>
+  <joint name="camera_init_joint" type="fixed">
+    <parent link="base_link"/>
+    <child link="camera_init"/>
+    <origin xyz="0.0 0.0 0.0" rpy="0 0 0"/>
+  </joint>
+  <link name="lidar_link"/>
+  <joint name="lidar_link_joint" type="fixed">
+    <parent link="base_link"/>
+    <child link="lidar_link"/>
+    <origin xyz="0.0 0.0 0.0" rpy="0 0 0"/>
+  </joint>
 </robot>

File: linorobot2_description/urdf/sensors/lidar.xacro (robot description, xacro)
@@ -1,93 +1,10 @@
-<?xml version="1.0"?>
-<robot xmlns:xacro="http://www.ros.org/wiki/xacro" >
-    <joint name="lidar_base_joint" type="fixed">
-        <parent link="base_link"/>
-        <child link="lidar_link"/>
-        <origin xyz="0.0 0 0.18" rpy="0 0 0"/>
-    </joint>
-    <link name="lidar_link">
-        <visual>
-            <geometry>
-                <cylinder radius="0.04267" length="0.05867"/>
-            </geometry>
-            <material name="red"/>
-        </visual>
-        <collision>
-            <geometry>
-                <cylinder radius="0.04267" length="0.05867"/>
-            </geometry>
-        </collision>
-        <cylinder mass="1.2" length="0.05867" radius="0.04267">
-            <origin xyz="0 0 0" rpy="0 0 0"/>
-        </cylinder>
-    </link>
-    <gazebo reference="lidar_link">
-        <material>Gazebo/Red</material>
-    </gazebo>
-    <joint name="laser_joint" type="fixed">
-        <parent link="lidar_link"/>
-        <child link="top"/>
-        <origin xyz="0 0 0.067" rpy="0 0 0"/>
-    </joint>
-    <link name="top">
-        <visual>
-            <geometry>
-                <cylinder radius="0.04267" length="0.07357"/>
-            </geometry>
-            <material name="red"/>
-        </visual>
-        <collision>
-            <geometry>
-                <cylinder radius="0.04267" length="0.07357"/>
-            </geometry>
-        </collision>
-        <cylinder mass="0.1" length="0.07357" radius="0.04267">
-            <origin xyz="0 0 0" rpy="0 0 0"/>
-        </cylinder>
-    </link>
-    <gazebo reference="lidar_link">
-        <material>Gazebo/Red</material>
-        <sensor type="ray" name="velodyne2-HDL32E">
-          <pose>0 0 0 0 0 0</pose>
-          <visualize>false</visualize>
-          <update_rate>10</update_rate>
-          <ray>
-                <scan>
-                    <horizontal>
-                        <samples>220</samples>
-                        <resolution>1</resolution>
-                        <min_angle>-3.142</min_angle>
-                        <max_angle>3.142</max_angle>
-                    </horizontal>
-                    <vertical>
-                        <samples>32</samples>
-                        <resolution>1</resolution>
-                        <min_angle>-0.535</min_angle>
-                        <max_angle> 0.186</max_angle>
-                    </vertical>
-                </scan>
-                <range>
-                    <min>0.3</min>
-                    <max>131.0</max>
-                    <resolution>0.001</resolution>
-                </range>
-                <noise>
-                    <type>gaussian</type>
-                    <mean>0.0</mean>
-                    <stddev>0.0</stddev>
-                </noise>
-          </ray>
-          <plugin name="gazebo_ros_laser_controller" filename="libgazebo_ros_velodyne_laser.so">
-            <ros>
-              <namespace>/velodyne2</namespace>
-              <remapping>~/out:=velodyne_points2</remapping>
-            </ros>
-            <frame_name>lidar_link</frame_name>
-            <organize_cloud>false</organize_cloud>
-            <min_range>0.9</min_range>
-            <max_range>130.0</max_range>
-            <gaussian_noise>0.008</gaussian_noise>
-          </plugin>
-        </sensor>
-    </gazebo>
+<robot xmlns:xacro="http://www.ros.org/wiki/xacro" name="vlp16">
+  <xacro:arg name="gpu" default="false"/>
+  <xacro:property name="gpu" value="$(arg gpu)" />
+  <xacro:arg name="organize_cloud" default="false"/>
+  <xacro:property name="organize_cloud" value="$(arg organize_cloud)" />
+  <xacro:include filename="$(find velodyne_description)/urdf/VLP-16.urdf.xacro"/>
+  <xacro:VLP-16 parent="base_link" name="velodyne" topic="/velodyne_points" organize_cloud="${organize_cloud}" hz="10" samples="440" gpu="${gpu}">
+    <origin xyz="0 0 0.0" rpy="0 0 0" />
+  </xacro:VLP-16>
 </robot>

Commit message: odom 을 중복으로 발행하고있어서 liosam실행시 위 아래로 진동하는 것!

File: linorobot2_description/urdf/controllers/skid_steer.urdf.xacro (robot description, xacro)
@@ -18,8 +18,8 @@
         <max_wheel_acceleration>1.0</max_wheel_acceleration>
         <robot_base_frame>base_link</robot_base_frame>
-        <publish_odom>false</publish_odom>
+        <publish_odom>true</publish_odom>
         <publish_odom_tf>false</publish_odom_tf>
         <publish_wheel_tf>false</publish_wheel_tf>
-        <odometry_frame>odom_gazebo</odometry_frame>
+        <odometry_frame>odom</odometry_frame>
       </plugin>
     </gazebo>

File: linorobot2_description/urdf/robots/4wd.urdf.xacro (robot description, xacro)
@@ -78,5 +78,5 @@
     wheel_torque="${wheel_torque}"
   />
-  <link name="camera_init"/>
+  <!-- <link name="camera_init"/>
   <joint name="camera_init_joint" type="fixed">
     <parent link="base_link"/>
@@ -89,4 +89,4 @@
     <child link="lidar_link"/>
     <origin xyz="0.0 0.0 0.0" rpy="0 0 0"/>
-  </joint>
+  </joint> -->
 </robot>
